Commit message: Update d435i.urdf.xacro

File: turtlebot_description/urdf/sensors/d435i.urdf.xacro (robot description, xacro)
@@ -32,5 +32,5 @@
     <!-- camera body, with origin at bottom screw mount -->
     <joint name="${name}_joint" type="fixed">
-    <origin xyz="${cam_px} 0.0205 ${cam_pz}" rpy="${cam_or} ${cam_op} ${cam_oy}"/>
+    <origin xyz="${cam_px} 0.0 ${cam_pz}" rpy="${cam_or} ${cam_op} ${cam_oy}"/>
       <parent link="${parent}"/>
       <child link="${name}_bottom_screw_frame" />
